Commit message: pull the drawer out

File: partnet-mobility-dataset/45290/mobility.urdf (robot description, URDF)
Before this commit: robot partnet_1d973f05e870af4b4da5feafe6f1c8fc, 5 links, 4 joints
Links:
- link link_0: mass None -> 0.1
- link link_1: mass None -> 0.1
- link link_2: mass None -> 0.1
- link link_3: mass None -> 0.5
